File: driver_40mm_atmega_v1p9/driver_40mm_atmega.kicad_pcb (KiCad board)
At the start: 6 copper layers, 40.4 x 40.4 mm, 424 parts, among them IC1 ATMEGA328P-M, IC2 ATMEGA328P-M, IC3 ATMEGA328P-M, IC4 ATMEGA328P-M, P1 CONN_2X2, P2 CONN_2X2, P3 CONN_2X2, P4 CONN_2X2, Q1 NMOS, Q10 NMOS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

Commit message: Some cleanup. Changed silkscreen to new v1.9.  Need to remake gerbers.
Other:
- board text added: "Panels G4 Driver V1.9R1"
- board text removed: "Panels G4 Driver V0.5 R1"
Changed lines of the file:
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@@
     (effects (font (size 1.016 1.016) (thickness 0.2032)) (justify mirror))
   )
-  (gr_text "Panels G4 Driver V0.5 R1" (at 50.94 70 90) (layer "B.SilkS")
+  (gr_text "Panels G4 Driver V1.9R1" (at 51 70 90) (layer "B.SilkS")
     (effects (font (size 1.016 1.016) (thickness 0.2032)) (justify mirror))
   )
