File: driver_40mm_atmega_v1p9/driver_40mm_atmega.kicad_sch (KiCad schematic)
At the start: 424 parts, among them IC1 ATMEGA328P-M, IC2 ATMEGA328P-M, IC3 ATMEGA328P-M, IC4 ATMEGA328P-M, P1 CONN_2X2, P2 CONN_2X2, P3 CONN_2X2, P4 CONN_2X2, Q1 NMOS, Q10 NMOS, Q11 NMOS, Q12 NMOS, Q13 NMOS, Q14 NMOS, Q15 NMOS, Q16 NMOS, Q2 NMOS, Q3 NMOS, Q4 NMOS, Q5 NMOS, Q6 NMOS, Q7 NMOS, Q8 NMOS, Q9 NMOS, X1 20MHz, X2 20MHz, X3 20MHz, X4 20MHz

Commit message: generate v1.9.3
Parts:
- C1, C2, C3, C37, C38, C39, C4, C40: Alt JLCPCB 01 (none) -> C1853386; Alt PN 01 (none) -> CC0201MRX5R6BB104; JLCPCB PN (none) -> C76937; PN (none) -> GRM033R61C104KE84D
- C10, C11, C12, C13, C14, C15, C16, C17, C18, C19, C20, C21, C22, C23, C24, C25, C26, C27, C28, C29, C30, C31, C32, C33, C34, C35, C36, C5, C6, C7, C8, C9: JLCPCB PN (none) -> C565508; PN (none) -> FN03B221K160PLG
- D1, D10, D100, D101, D102, D103, D104, D105, D106, D107, D108, D109, D11, D110, D111, D112, D113, D114, D115, D116, D117, D118, D119, D12, D120, D121, D122, D123, D124, D125, D126, D127, D128, D129, D13, D130, D131, D132, D133, D134, D135, D136, D137, D138, D139, D14, D140, D141, D142, D143, D144, D145, D146, D147, D148, D149, D15, D150, D151, D152, D153, D154, D155, D156, D157, D158, D159, D16, D160, D161, D162, D163, D164, D165, D166, D167, D168, D169, D17, D170, D171, D172, D173, D174, D175, D176, D177, D178, D179, D18, D180, D181, D182, D183, D184, D185, D186, D187, D188, D189, D19, D190, D191, D192, D193, D194, D195, D196, D197, D198, D199, D2, D20, D200, D201, D202, D203, D204, D205, D206, D207, D208, D209, D21, D210, D211, D212, D213, D214, D215, D216, D217, D218, D219, D22, D220, D221, D222, D223, D224, D225, D226, D227, D228, D229, D23, D230, D231, D232, D233, D234, D235, D236, D237, D238, D239, D24, D240, D241, D242, D243, D244, D245, D246, D247, D248, D249, D25, D250, D251, D252, D253, D254, D255, D256, D26, D27, D28, D29, D3, D30, D31, D32, D33, D34, D35, D36, D37, D38, D39, D4, D40, D41, D42, D43, D44, D45, D46, D47, D48, D49, D5, D50, D51, D52, D53, D54, D55, D56, D57, D58, D59, D6, D60, D61, D62, D63, D64, D65, D66, D67, D68, D69, D7, D70, D71, D72, D73, D74, D75, D76, D77, D78, D79, D8, D80, D81, D82, D83, D84, D85, D86, D87, D88, D89, D9, D90, D91, D92, D93, D94, D95, D96, D97, D98, D99: JLCPCB PN (none) -> C5160718; PN (none) -> A-SP136G2C-C01-3T
- IC1, IC2, IC3, IC4: JLCPCB PN (none) -> C2651951; PN (none) -> ATMEGA328P-MUR
- P1, P2, P3, P4: JLCPCB PN (none) -> C7499901; PN (none) -> TSM-102-01-L-DV-P-TR
- Q1, Q10, Q11, Q12, Q13, Q14, Q15, Q16, Q2, Q3, Q4, Q5, Q6, Q7, Q8, Q9: JLCPCB PN (none) -> C145239; PN (none) -> SI1034CX-T1-GE3
- R1, R2, R3, R4: JLCPCB PN (none) -> C226669; PN (none) -> AC0201JR-074K7L
- R10, R11, R12, R13, R14, R15, R16, R17, R18, R19, R20, R21, R22, R23, R24, R25, R26, R27, R28, R29, R30, R31, R32, R33, R34, R35, R36, R5, R6, R7, R8, R9: JLCPCB PN (none) -> C5141103; PN (none) -> SC0201F1800G1BNRH
- R100, R38, R40, R42, R44, R46, R48, R50, R52, R55, R56, R59, R60, R63, R64, R67, R68, R71, R72, R75, R76, R79, R80, R83, R84, R87, R88, R91, R92, R95, R96, R99: JLCPCB PN (none) -> C102689; PN (none) -> RTT01102JTH
- R37, R39, R41, R43, R45, R47, R49, R51, R53, R54, R57, R58, R61, R62, R65, R66, R69, R70, R73, R74, R77, R78, R81, R82, R85, R86, R89, R90, R93, R94, R97, R98: JLCPCB PN (none) -> C2991668; PN (none) -> RHC-01W1000FT
- X1, X2, X3, X4: JLCPCB PN (none) -> C882604; PN (none) -> CSTNE20M0V530000R0
Other:
- company: (none) -> Janelia
- title: (none) -> G4 Driver 40mm ATMega
